Commit message: add urdf.xacro file

File: workspace/src/av_description/urdf/autoVehi.urdf.xacro (robot description, xacro)
@@ -1,4 +1,14 @@
 <?xml version="1.0"?>
 <robot xmlns:xacro="http://www.ros.org/wiki/xacro" name="autoVehi">
-    <xacro:include filename="autoVehi_core.urdf.xacro" />
+    <xacro:property name="PI" value="3.1415926535897931"/>
+    <xacro:include filename="$(find av_description)/urdf/autoVehi_core.urdf.xacro" />
+    <link name="world"/>
+    <joint name="vitual_joint" type="fixed">
+        <parent link="world"/>
+        <child link="base_link"/>
+        <origin xyz="0 0 0" rpy="0 0 0"/>
+    </joint>
+    <xacro:autoVehi>
+        <origin xyz="0 0 0" rpy="0 0 0"/>
+    </xacro:autoVehi>
 </robot>

File: workspace/src/av_description/urdf/autoVehi_core.urdf.xacro (robot description, xacro)
@@ -1,3 +1,181 @@
 <?xml version="1.0"?>
 <robot xmlns:xacro="http://www.ros.org/wiki/xacro" name="autoVehi">
+    <xacro:property name="max_effort" value="300"/>
+    <xacro:property name="joint_damping" value="0.5"/>
+    <xacro:macro name="autoVehi" params=" *origin">
+        <material name="white">
+            <color rgba=" 1 1 1 0.5"/>
+        </material>
+        <material name="blue">
+            <color rgba="0.1 0.1 1 0.5"/>
+        </material>
+        <material name="red">
+            <color rgba="1 0.1 0.1 0.5"/>
+        </material>
+        <material name="green">
+            <color rgba="0.1 1 0.1 0.5"/>
+        </material>
+        <link name="base_link"></link>
+        <joint name="chassis_joint" type="fixed">
+            <parent link="base_link"/>
+            <child link="chassis_link"/>
+            <origin xyz="0.5 0 0.15"/>
+        </joint>
+        <link name="chassis_link">
+            <inertial>
+                <origin xyz="0 0 0.15" rpy="0 0 0"/>
+                <mass value="20"/>
+                <inertia
+                    ixx="0.566" ixy="0" ixz="0"
+                    iyy="1.816" iyz="0"
+                    izz="2.083"/>
+            </inertial>
+            <visual>
+                <origin xyz="0 0 0.15" rpy="0 0 0"/>
+                <geometry>
+                    <box size="1 0.5 0.3"/>
+                </geometry>
+                <material name="white"/>
+            </visual>
+            <collision>
+                <origin xyz="0 0 0.15" rpy="0 0 0"/>
+                <geometry>
+                    <box size="1 0.5 0.3"/>
+                </geometry>
+                <material name="white"/>
+            </collision>
+        </link>
+        <!--/////////////// wheel_left_top////////////-->
+        <joint name="wheel_left_top_joint" type="continuous">
+            <parent link="chassis_link"/>
+            <child link="wheel_left_top" />
+            <origin xyz="0.3 0.25 0" rpy="${-PI/2} 0 0"/>
+            <axis xyz="0 0 1"/>
+            <limit effort="${max_effort}" velocity="${PI}"/>
+            <dynamics damping="${joint_damping}"/>
+        </joint>
+        <link name="wheel_left_top">
+            <inertial>
+                <origin xyz="0 0 0.05" rpy="0 0 0"/>
+                <mass value="1"/>
+                <inertia
+                    ixx="0.006" ixy="0" ixz="0"
+                    iyy="0.006" iyz="0"
+                    izz="0.011"/>
+            </inertial>
+            <visual>
+                <origin xyz="0 0 0.05" rpy="0 0 0"/>
+                <geometry>
+                    <cylinder radius="0.15" length="0.1"/>
+                </geometry>
+                <material name="green"/>
+            </visual>
+            <collision>
+                <origin xyz="0 0 0.05" rpy="0 0 0"/>
+                <geometry>
+                    <cylinder radius="0.15" length="0.1"/>
+                </geometry>
+                <material name="green"/>
+            </collision>
+        </link>
+        <!--/////////////// wheel_left_bot////////////-->
+        <joint name="wheel_left_bot_joint" type="continuous">
+            <parent link="chassis_link"/>
+            <child link="wheel_left_bot" />
+            <origin xyz="-0.3 0.25 0" rpy="${-PI/2} 0 0"/>
+            <axis xyz="0 0 1"/>
+            <limit effort="${max_effort}" velocity="${PI}"/>
+            <dynamics damping="${joint_damping}"/>
+        </joint>
+        <link name="wheel_left_bot">
+            <inertial>
+                <origin xyz="0 0 0.05" rpy="0 0 0"/>
+                <mass value="1"/>
+                <inertia
+                    ixx="0.006" ixy="0" ixz="0"
+                    iyy="0.006" iyz="0"
+                    izz="0.011"/>
+            </inertial>
+            <visual>
+                <origin xyz="0 0 0.05" rpy="0 0 0"/>
+                <geometry>
+                    <cylinder radius="0.15" length="0.1"/>
+                </geometry>
+                <material name="green"/>
+            </visual>
+            <collision>
+                <origin xyz="0 0 0.05" rpy="0 0 0"/>
+                <geometry>
+                    <cylinder radius="0.15" length="0.1"/>
+                </geometry>
+                <material name="green"/>
+            </collision>
+        </link>
+        <!--/////////////// wheel_right_top////////////-->
+        <joint name="wheel_right_top_joint" type="continuous">
+            <parent link="chassis_link"/>
+            <child link="wheel_right_top" />
+            <origin xyz="0.3 -0.25 0" rpy="${PI/2} 0 0"/>
+            <axis xyz="0 0 1"/>
+            <limit effort="${max_effort}" velocity="${PI}"/>
+            <dynamics damping="${joint_damping}"/>
+        </joint>
+        <link name="wheel_right_top">
+            <inertial>
+                <origin xyz="0 0 0.05" rpy="0 0 0"/>
+                <mass value="1"/>
+                <inertia
+                    ixx="0.006" ixy="0" ixz="0"
+                    iyy="0.006" iyz="0"
+                    izz="0.011"/>
+            </inertial>
+            <visual>
+                <origin xyz="0 0 0.05" rpy="0 0 0"/>
+                <geometry>
+                    <cylinder radius="0.15" length="0.1"/>
+                </geometry>
+                <material name="green"/>
+            </visual>
+            <collision>
+                <origin xyz="0 0 0.05" rpy="0 0 0"/>
+                <geometry>
+                    <cylinder radius="0.15" length="0.1"/>
+                </geometry>
+                <material name="green"/>
+            </collision>
+        </link>
+        <!--/////////////// wheel_right_bot////////////-->
+        <joint name="wheel_right_bot_joint" type="continuous">
+            <parent link="chassis_link"/>
+            <child link="wheel_right_bot" />
+            <origin xyz="-0.3 -0.25 0" rpy="${PI/2} 0 0"/>
+            <axis xyz="0 0 1"/>
+            <limit effort="${max_effort}" velocity="${PI}"/>
+            <dynamics damping="${joint_damping}"/>
+        </joint>
+        <link name="wheel_right_bot">
+            <inertial>
+                <origin xyz="0 0 0.05" rpy="0 0 0"/>
+                <mass value="1"/>
+                <inertia
+                    ixx="0.006" ixy="0" ixz="0"
+                    iyy="0.006" iyz="0"
+                    izz="0.011"/>
+            </inertial>
+            <visual>
+                <origin xyz="0 0 0.05" rpy="0 0 0"/>
+                <geometry>
+                    <cylinder radius="0.15" length="0.1"/>
+                </geometry>
+                <material name="green"/>
+            </visual>
+            <collision>
+                <origin xyz="0 0 0.05" rpy="0 0 0"/>
+                <geometry>
+                    <cylinder radius="0.15" length="0.1"/>
+                </geometry>
+                <material name="green"/>
+            </collision>
+        </link>
+    </xacro:macro>
 </robot>

Commit message: add gazebo

File: workspace/src/av_description/urdf/autoVehi.urdf.xacro (robot description, xacro)
@@ -2,7 +2,9 @@
 <robot xmlns:xacro="http://www.ros.org/wiki/xacro" name="autoVehi">
     <xacro:property name="PI" value="3.1415926535897931"/>
+    <xacro:arg name="robot_name" default="autoVehi"/>
+    <xacro:arg name="use_gazebo" default="false"/>
     <xacro:include filename="$(find av_description)/urdf/autoVehi_core.urdf.xacro" />
     <link name="world"/>
-    <joint name="vitual_joint" type="fixed">
+    <joint name="virtual_joint" type="fixed">
         <parent link="world"/>
         <child link="base_link"/>
@@ -12,3 +14,10 @@
         <origin xyz="0 0 0" rpy="0 0 0"/>
     </xacro:autoVehi>
+    <xacro:include filename="$(find av_description)/urdf/control/gazebo_sim_ros2_control.urdf.xacro" />
+    <xacro:load_gazebo_sim_ros2_control_plugin
+        robot_name="$(arg robot_name)"
+        use_gazebo="$(arg use_gazebo)"/>
+    <xacro:include filename="$(find av_description)/urdf/control/autoVehi_ros2_control.urdf.xacro" />
+    <xacro:av_ros2_control
+        use_gazebo="$(arg use_gazebo)"/>
 </robot>

Commit message: add models

File: workspace/src/av_description/urdf/autoVehi.urdf.xacro (robot description, xacro)
@@ -4,5 +4,8 @@
     <xacro:arg name="robot_name" default="autoVehi"/>
     <xacro:arg name="use_gazebo" default="false"/>
+    <xacro:arg name="prefix" default=""/>
     <xacro:include filename="$(find av_description)/urdf/autoVehi_core.urdf.xacro" />
+    <xacro:autoVehi/>
+<!--
     <link name="world"/>
     <joint name="virtual_joint" type="fixed">
@@ -10,8 +13,30 @@
         <child link="base_link"/>
         <origin xyz="0 0 0" rpy="0 0 0"/>
-    </joint>
-    <xacro:autoVehi>
-        <origin xyz="0 0 0" rpy="0 0 0"/>
-    </xacro:autoVehi>
+    </joint> -->
+    <xacro:include filename="$(find av_description)/urdf/sensor/imu.urdf.xacro"/>
+    <xacro:imu_sensor
+      prefix="$(arg prefix)"
+      parent="chassis_link"
+      frame_id="imu"
+      xyz_offset="0 0 0"
+      rpy_offset="0 0 0"
+      update_rate="15.0"
+      topic_name="imu/data"/>
+    <xacro:include filename="$(find av_description)/urdf/sensor/lidar.urdf.xacro"/>
+    <xacro:lidar_sensor
+      prefix="$(arg prefix)"
+      parent="chassis_link"
+      frame_id="laser_frame"
+      xyz_offset="0.5 0 0.3"
+      rpy_offset="0 0 0"
+      mesh_xyz_offset="0 0 0.02"
+      mesh_rpy_offset="0 0 0"
+      topic_name="scan"/>
+    <xacro:include filename="$(find av_description)/urdf/sensor/camera.urdf.xacro"/>
+    <xacro:camera
+      prefix="$(arg prefix)"
+      camera_name="cam_1"
+      xyz_offset="0.5 0 0.15"
+      rpy_offset="0 0 0"/>
     <xacro:include filename="$(find av_description)/urdf/control/gazebo_sim_ros2_control.urdf.xacro" />
     <xacro:load_gazebo_sim_ros2_control_plugin

File: workspace/src/av_description/urdf/autoVehi_core.urdf.xacro (robot description, xacro)
@@ -3,5 +3,5 @@
     <xacro:property name="max_effort" value="300"/>
     <xacro:property name="joint_damping" value="0.5"/>
-    <xacro:macro name="autoVehi" params=" *origin">
+    <xacro:macro name="autoVehi" params="">
         <material name="white">
             <color rgba=" 1 1 1 0.5"/>
@@ -14,5 +14,5 @@
         </material>
         <material name="green">
-            <color rgba="0.1 1 0.1 0.5"/>
+            <color rgba="0.1 1 0.1 0.8"/>
         </material>
         <link name="base_link"></link>
@@ -20,5 +20,5 @@
             <parent link="base_link"/>
             <child link="chassis_link"/>
-            <origin xyz="0.5 0 0.15"/>
+            <origin xyz="0 0 0.15"/>
         </joint>
         <link name="chassis_link">
@@ -43,5 +43,4 @@
                     <box size="1 0.5 0.3"/>
                 </geometry>
-                <material name="white"/>
             </collision>
         </link>
@@ -76,5 +75,4 @@
                     <cylinder radius="0.15" length="0.1"/>
                 </geometry>
-                <material name="green"/>
             </collision>
         </link>
@@ -109,5 +107,4 @@
                     <cylinder radius="0.15" length="0.1"/>
                 </geometry>
-                <material name="green"/>
             </collision>
         </link>
@@ -142,5 +139,4 @@
                     <cylinder radius="0.15" length="0.1"/>
                 </geometry>
-                <material name="green"/>
             </collision>
         </link>
@@ -175,7 +171,58 @@
                     <cylinder radius="0.15" length="0.1"/>
                 </geometry>
-                <material name="green"/>
-            </collision>
-        </link>
+            </collision>
+        </link>
+        <gazebo reference="wheel_left_top">
+            <collision>
+                <surface>
+                    <friction>
+                        <ode>
+                            <mu>0.0</mu>
+                            <mu2>0.0</mu2>
+                            <minDepth>0.001</minDepth>
+                        </ode>
+                    </friction>
+                </surface>
+            </collision>
+        </gazebo>
+        <gazebo reference="wheel_left_bot">
+            <collision>
+                <surface>
+                    <friction>
+                        <ode>
+                            <mu>1.0</mu>
+                            <mu2>1.0</mu2>
+                            <minDepth>0.001</minDepth>
+                        </ode>
+                    </friction>
+                </surface>
+            </collision>
+        </gazebo>
+        <gazebo reference="wheel_right_top">
+            <collision>
+                <surface>
+                    <friction>
+                        <ode>
+                            <mu>0.0</mu>
+                            <mu2>0.0</mu2>
+                            <minDepth>0.001</minDepth>
+                        </ode>
+                    </friction>
+                </surface>
+            </collision>
+        </gazebo>
+        <gazebo reference="wheel_right_bot">
+            <collision>
+                <surface>
+                    <friction>
+                        <ode>
+                            <mu>1.0</mu>
+                            <mu2>1.0</mu2>
+                            <minDepth>0.001</minDepth>
+                        </ode>
+                    </friction>
+                </surface>
+            </collision>
+        </gazebo>
     </xacro:macro>
 </robot>
