Commit message: add gazebo workspace

File: workspace/src/av_description/urdf/autoVehi_core.urdf.xacro (robot description, xacro)
@@ -117,5 +117,5 @@
             <child link="wheel_right_top" />
             <origin xyz="0.3 -0.25 0" rpy="${PI/2} 0 0"/>
-            <axis xyz="0 0 1"/>
+            <axis xyz="0 0 -1"/>
             <limit effort="${max_effort}" velocity="${PI}"/>
             <dynamics damping="${joint_damping}"/>
@@ -150,5 +150,5 @@
             <child link="wheel_right_bot" />
             <origin xyz="-0.3 -0.25 0" rpy="${PI/2} 0 0"/>
-            <axis xyz="0 0 1"/>
+            <axis xyz="0 0 -1"/>
             <limit effort="${max_effort}" velocity="${PI}"/>
             <dynamics damping="${joint_damping}"/>

Commit message: fix inertial

File: workspace/src/av_description/urdf/autoVehi_core.urdf.xacro (robot description, xacro)
@@ -16,4 +16,7 @@
             <color rgba="0.1 1 0.1 0.8"/>
         </material>
+        <material name="black">
+            <color rgba="1 1 1 0.8"/>
+        </material>
         <link name="base_link"></link>
         <joint name="chassis_joint" type="fixed">
@@ -36,5 +39,5 @@
                     <box size="1 0.5 0.3"/>
                 </geometry>
-                <material name="white"/>
+                <material name="blue"/>
             </visual>
             <collision>
@@ -56,20 +59,20 @@
         <link name="wheel_left_top">
             <inertial>
-                <origin xyz="0 0 0.05" rpy="0 0 0"/>
-                <mass value="1"/>
-                <inertia
-                    ixx="0.006" ixy="0" ixz="0"
-                    iyy="0.006" iyz="0"
-                    izz="0.011"/>
-            </inertial>
-            <visual>
-                <origin xyz="0 0 0.05" rpy="0 0 0"/>
-                <geometry>
-                    <cylinder radius="0.15" length="0.1"/>
-                </geometry>
-                <material name="green"/>
-            </visual>
-            <collision>
-                <origin xyz="0 0 0.05" rpy="0 0 0"/>
+                <origin xyz="0 0 0.06" rpy="0 0 0"/>
+                <mass value="1"/>
+                <inertia
+                    ixx="0.006" ixy="0" ixz="0"
+                    iyy="0.006" iyz="0"
+                    izz="0.011"/>
+            </inertial>
+            <visual>
+                <origin xyz="0 0 0.06" rpy="0 0 0"/>
+                <geometry>
+                    <cylinder radius="0.15" length="0.1"/>
+                </geometry>
+                <material name="black"/>
+            </visual>
+            <collision>
+                <origin xyz="0 0 0.06" rpy="0 0 0"/>
                 <geometry>
                     <cylinder radius="0.15" length="0.1"/>
@@ -88,20 +91,20 @@
         <link name="wheel_left_bot">
             <inertial>
-                <origin xyz="0 0 0.05" rpy="0 0 0"/>
-                <mass value="1"/>
-                <inertia
-                    ixx="0.006" ixy="0" ixz="0"
-                    iyy="0.006" iyz="0"
-                    izz="0.011"/>
-            </inertial>
-            <visual>
-                <origin xyz="0 0 0.05" rpy="0 0 0"/>
-                <geometry>
-                    <cylinder radius="0.15" length="0.1"/>
-                </geometry>
-                <material name="green"/>
-            </visual>
-            <collision>
-                <origin xyz="0 0 0.05" rpy="0 0 0"/>
+                <origin xyz="0 0 0.06" rpy="0 0 0"/>
+                <mass value="1"/>
+                <inertia
+                    ixx="0.006" ixy="0" ixz="0"
+                    iyy="0.006" iyz="0"
+                    izz="0.011"/>
+            </inertial>
+            <visual>
+                <origin xyz="0 0 0.06" rpy="0 0 0"/>
+                <geometry>
+                    <cylinder radius="0.15" length="0.1"/>
+                </geometry>
+                <material name="black"/>
+            </visual>
+            <collision>
+                <origin xyz="0 0 0.06" rpy="0 0 0"/>
                 <geometry>
                     <cylinder radius="0.15" length="0.1"/>
@@ -120,20 +123,20 @@
         <link name="wheel_right_top">
             <inertial>
-                <origin xyz="0 0 0.05" rpy="0 0 0"/>
-                <mass value="1"/>
-                <inertia
-                    ixx="0.006" ixy="0" ixz="0"
-                    iyy="0.006" iyz="0"
-                    izz="0.011"/>
-            </inertial>
-            <visual>
-                <origin xyz="0 0 0.05" rpy="0 0 0"/>
-                <geometry>
-                    <cylinder radius="0.15" length="0.1"/>
-                </geometry>
-                <material name="green"/>
-            </visual>
-            <collision>
-                <origin xyz="0 0 0.05" rpy="0 0 0"/>
+                <origin xyz="0 0 0.06" rpy="0 0 0"/>
+                <mass value="1"/>
+                <inertia
+                    ixx="0.006" ixy="0" ixz="0"
+                    iyy="0.006" iyz="0"
+                    izz="0.011"/>
+            </inertial>
+            <visual>
+                <origin xyz="0 0 0.06" rpy="0 0 0"/>
+                <geometry>
+                    <cylinder radius="0.15" length="0.1"/>
+                </geometry>
+                <material name="black"/>
+            </visual>
+            <collision>
+                <origin xyz="0 0 0.06" rpy="0 0 0"/>
                 <geometry>
                     <cylinder radius="0.15" length="0.1"/>
@@ -152,20 +155,20 @@
         <link name="wheel_right_bot">
             <inertial>
-                <origin xyz="0 0 0.05" rpy="0 0 0"/>
-                <mass value="1"/>
-                <inertia
-                    ixx="0.006" ixy="0" ixz="0"
-                    iyy="0.006" iyz="0"
-                    izz="0.011"/>
-            </inertial>
-            <visual>
-                <origin xyz="0 0 0.05" rpy="0 0 0"/>
-                <geometry>
-                    <cylinder radius="0.15" length="0.1"/>
-                </geometry>
-                <material name="green"/>
-            </visual>
-            <collision>
-                <origin xyz="0 0 0.05" rpy="0 0 0"/>
+                <origin xyz="0 0 0.06" rpy="0 0 0"/>
+                <mass value="1"/>
+                <inertia
+                    ixx="0.006" ixy="0" ixz="0"
+                    iyy="0.006" iyz="0"
+                    izz="0.011"/>
+            </inertial>
+            <visual>
+                <origin xyz="0 0 0.06" rpy="0 0 0"/>
+                <geometry>
+                    <cylinder radius="0.15" length="0.1"/>
+                </geometry>
+                <material name="black"/>
+            </visual>
+            <collision>
+                <origin xyz="0 0 0.06" rpy="0 0 0"/>
                 <geometry>
                     <cylinder radius="0.15" length="0.1"/>

Commit message: camera

File: workspace/src/av_description/urdf/autoVehi_core.urdf.xacro (robot description, xacro)
@@ -59,20 +59,20 @@
         <link name="wheel_left_top">
             <inertial>
-                <origin xyz="0 0 0.06" rpy="0 0 0"/>
-                <mass value="1"/>
-                <inertia
-                    ixx="0.006" ixy="0" ixz="0"
-                    iyy="0.006" iyz="0"
-                    izz="0.011"/>
-            </inertial>
-            <visual>
-                <origin xyz="0 0 0.06" rpy="0 0 0"/>
-                <geometry>
-                    <cylinder radius="0.15" length="0.1"/>
-                </geometry>
-                <material name="black"/>
-            </visual>
-            <collision>
-                <origin xyz="0 0 0.06" rpy="0 0 0"/>
+                <origin xyz="0 0 0.05" rpy="0 0 0"/>
+                <mass value="1"/>
+                <inertia
+                    ixx="0.006" ixy="0" ixz="0"
+                    iyy="0.006" iyz="0"
+                    izz="0.011"/>
+            </inertial>
+            <visual>
+                <origin xyz="0 0 0.05" rpy="0 0 0"/>
+                <geometry>
+                    <cylinder radius="0.15" length="0.1"/>
+                </geometry>
+                <material name="black"/>
+            </visual>
+            <collision>
+                <origin xyz="0 0 0.05" rpy="0 0 0"/>
                 <geometry>
                     <cylinder radius="0.15" length="0.1"/>
@@ -91,20 +91,20 @@
         <link name="wheel_left_bot">
             <inertial>
-                <origin xyz="0 0 0.06" rpy="0 0 0"/>
-                <mass value="1"/>
-                <inertia
-                    ixx="0.006" ixy="0" ixz="0"
-                    iyy="0.006" iyz="0"
-                    izz="0.011"/>
-            </inertial>
-            <visual>
-                <origin xyz="0 0 0.06" rpy="0 0 0"/>
-                <geometry>
-                    <cylinder radius="0.15" length="0.1"/>
-                </geometry>
-                <material name="black"/>
-            </visual>
-            <collision>
-                <origin xyz="0 0 0.06" rpy="0 0 0"/>
+                <origin xyz="0 0 0.05" rpy="0 0 0"/>
+                <mass value="1"/>
+                <inertia
+                    ixx="0.006" ixy="0" ixz="0"
+                    iyy="0.006" iyz="0"
+                    izz="0.011"/>
+            </inertial>
+            <visual>
+                <origin xyz="0 0 0.05" rpy="0 0 0"/>
+                <geometry>
+                    <cylinder radius="0.15" length="0.1"/>
+                </geometry>
+                <material name="black"/>
+            </visual>
+            <collision>
+                <origin xyz="0 0 0.05" rpy="0 0 0"/>
                 <geometry>
                     <cylinder radius="0.15" length="0.1"/>
@@ -123,20 +123,20 @@
         <link name="wheel_right_top">
             <inertial>
-                <origin xyz="0 0 0.06" rpy="0 0 0"/>
-                <mass value="1"/>
-                <inertia
-                    ixx="0.006" ixy="0" ixz="0"
-                    iyy="0.006" iyz="0"
-                    izz="0.011"/>
-            </inertial>
-            <visual>
-                <origin xyz="0 0 0.06" rpy="0 0 0"/>
-                <geometry>
-                    <cylinder radius="0.15" length="0.1"/>
-                </geometry>
-                <material name="black"/>
-            </visual>
-            <collision>
-                <origin xyz="0 0 0.06" rpy="0 0 0"/>
+                <origin xyz="0 0 0.05" rpy="0 0 0"/>
+                <mass value="1"/>
+                <inertia
+                    ixx="0.006" ixy="0" ixz="0"
+                    iyy="0.006" iyz="0"
+                    izz="0.011"/>
+            </inertial>
+            <visual>
+                <origin xyz="0 0 0.05" rpy="0 0 0"/>
+                <geometry>
+                    <cylinder radius="0.15" length="0.1"/>
+                </geometry>
+                <material name="black"/>
+            </visual>
+            <collision>
+                <origin xyz="0 0 0.05" rpy="0 0 0"/>
                 <geometry>
                     <cylinder radius="0.15" length="0.1"/>
@@ -155,20 +155,20 @@
         <link name="wheel_right_bot">
             <inertial>
-                <origin xyz="0 0 0.06" rpy="0 0 0"/>
-                <mass value="1"/>
-                <inertia
-                    ixx="0.006" ixy="0" ixz="0"
-                    iyy="0.006" iyz="0"
-                    izz="0.011"/>
-            </inertial>
-            <visual>
-                <origin xyz="0 0 0.06" rpy="0 0 0"/>
-                <geometry>
-                    <cylinder radius="0.15" length="0.1"/>
-                </geometry>
-                <material name="black"/>
-            </visual>
-            <collision>
-                <origin xyz="0 0 0.06" rpy="0 0 0"/>
+                <origin xyz="0 0 0.05" rpy="0 0 0"/>
+                <mass value="1"/>
+                <inertia
+                    ixx="0.006" ixy="0" ixz="0"
+                    iyy="0.006" iyz="0"
+                    izz="0.011"/>
+            </inertial>
+            <visual>
+                <origin xyz="0 0 0.05" rpy="0 0 0"/>
+                <geometry>
+                    <cylinder radius="0.15" length="0.1"/>
+                </geometry>
+                <material name="black"/>
+            </visual>
+            <collision>
+                <origin xyz="0 0 0.05" rpy="0 0 0"/>
                 <geometry>
                     <cylinder radius="0.15" length="0.1"/>
@@ -183,5 +183,4 @@
                             <mu>0.0</mu>
                             <mu2>0.0</mu2>
-                            <minDepth>0.001</minDepth>
                         </ode>
                     </friction>
@@ -196,5 +195,4 @@
                             <mu>1.0</mu>
                             <mu2>1.0</mu2>
-                            <minDepth>0.001</minDepth>
                         </ode>
                     </friction>
@@ -209,5 +207,4 @@
                             <mu>0.0</mu>
                             <mu2>0.0</mu2>
-                            <minDepth>0.001</minDepth>
                         </ode>
                     </friction>
@@ -222,5 +219,4 @@
                             <mu>1.0</mu>
                             <mu2>1.0</mu2>
-                            <minDepth>0.001</minDepth>
                         </ode>
                     </friction>

File: workspace/src/av_description/urdf/sensor/camera.urdf.xacro (robot description, xacro)
@@ -34,6 +34,6 @@
     image_height:=240
     clip_near:=0.05
-    clip_far:=1.5
-    update_rate:=2
+    clip_far:=10
+    update_rate:=10
     always_on:=1
     visualize:=true">
@@ -94,5 +94,5 @@
         <always_on>${always_on}</always_on>
         <gz_frame_id>${prefix}${camera_name}_color_optical_frame</gz_frame_id>
-        <topic>${camera_name}</topic>
+        <topic>${camera_name}/image</topic>
         <update_rate>${update_rate}</update_rate>
         <visualize>${visualize}</visualize>
